File: pcb/keyboard6.kicad_pcb (KiCad board)
At the start: 2 copper layers, 149.9 x 129.4 mm, 80 parts, among them J1 AudioJack4, J2 USB_B_Micro, SW1 SW_DIP_x01, SW10 SW_DIP_x01, SW11 SW_DIP_x01, SW12 SW_DIP_x01, SW13 SW_DIP_x01, SW14 SW_DIP_x01, SW15 SW_DIP_x01, SW16 SW_DIP_x01, SW17 SW_DIP_x01, SW18 SW_DIP_x01, SW19 SW_DIP_x01, SW2 SW_DIP_x01, SW20 SW_DIP_x01, SW21 SW_DIP_x01, SW22 SW_DIP_x01, SW23 SW_DIP_x01, SW24 SW_DIP_x01, SW25 SW_DIP_x01, SW26 SW_DIP_x01, SW27 SW_DIP_x01, SW28 SW_DIP_x01, SW29 SW_DIP_x01, SW3 SW_DIP_x01, SW30 SW_Push_Dual, SW4 SW_DIP_x01, SW5 SW_DIP_x01, SW6 SW_DIP_x01, SW7 SW_DIP_x01, SW8 SW_DIP_x01, SW9 SW_DIP_x01, Y1 16MHz

Commit message: minor change.
Parts:
- moved J2 0.60 mm to (-24.6, -10.5)
Other:
- board size 149.9 x 129.4 mm -> 150.9 x 130.2 mm

Commit message: All routed.
Parts:
- SW1, SW10, SW11, SW12, SW13, SW14, SW15, SW16, SW17, SW18, SW19, SW2, SW20, SW21, SW22, SW23, SW24, SW25, SW26, SW27, SW28, SW29, SW3, SW4, SW5, SW6, SW7, SW8, SW9: moved to B.Cu
- moved D29 5.74 mm to (-32.0, 24.1)
- moved D15 5.20 mm to (60.5, 0.00), turned to 270 degrees
- moved D16 5.20 mm to (60.5, -19.1), turned to 270 degrees
- moved D17 5.20 mm to (60.5, -38.2), turned to 270 degrees
- moved D18 5.20 mm to (60.5, -57.3), turned to 270 degrees
- moved D19 5.20 mm to (60.5, -76.4), turned to 270 degrees
- moved D24 5.20 mm to (98.7, -19.1), turned to 270 degrees
- moved D25 5.20 mm to (98.7, -38.2), turned to 270 degrees
- moved D26 5.20 mm to (98.7, 34.4), turned to 270 degrees
- moved D1 5.20 mm to (3.20, -15.1), turned to 270 degrees
- moved D2 5.20 mm to (3.20, -34.2), turned to 270 degrees
- moved D3 5.20 mm to (3.20, -53.3), turned to 270 degrees
- moved D4 5.20 mm to (3.20, -72.4), turned to 270 degrees
- moved D5 5.20 mm to (22.3, 0.00), turned to 270 degrees
- moved D6 5.20 mm to (22.3, -19.1), turned to 270 degrees
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Connections:
- C2 pad 2: Net-(C2-Pad2) -> GND1
- C3 pad 2: Net-(C2-Pad2) -> GND1
- C4 pad 2: Net-(C2-Pad2) -> GND1
Routing:
- net GND1: track 0.00 -> 57.4 mm, vias 0 -> 24
- net /Controller/col1: track 135.7 -> 175.9 mm, vias 2 -> 0
- net /Controller/col5: track 116.6 -> 98.1 mm
- net /Controller/col4: track 132.1 -> 113.7 mm
- net /Controller/row3: track 253.3 -> 271.5 mm, vias 12 -> 10
- net /Controller/col3: track 150.2 -> 136.5 mm
- net /Controller/row0: track 279.3 -> 268.1 mm
- net /Controller/row1: track 228.9 -> 238.6 mm, vias 8 -> 10
- net /Controller/col2: track 143.7 -> 152.8 mm
- net /Controller/row2: track 210.5 -> 219.0 mm, vias 12 -> 10
- net Net-(D28-Pad1): track 5.25 -> 12.9 mm
- net Net-(D27-Pad1): track 9.66 -> 3.39 mm
- net Net-(D8-Pad1): track 0.00 -> 5.54 mm
- net Net-(D7-Pad1): track 0.00 -> 5.54 mm
- net Net-(D11-Pad1): track 0.00 -> 5.54 mm
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- added copper zone on B.Cu, net GND1
Other:
- net class Default: clearance 0.2 -> 0.3
- rule trace_clearance: 0.2 -> 0.3

Commit message: drc clean
Other:
- net class Default: clearance 0.3 -> 0.25
- rule trace_clearance: 0.3 -> 0.25

Commit message: add soldermask clearance.
Other:
- rule pad_to_mask_clearance: 0 -> 0.05
Changed lines of the file:
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@@
     (pad_size 4 4)
     (pad_drill 4)
-    (pad_to_mask_clearance 0)
+    (pad_to_mask_clearance 0.05)
     (aux_axis_origin 0 0)
     (visible_elements FFFFFFFF)

Commit message: minor change
Parts:
- C1, C5: value 16p -> 32p
Changed lines of the file:
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@@
       (effects (font (size 1 1) (thickness 0.15)))
     )
-    (fp_text value 16p (at 0 1.68) (layer F.Fab)
+    (fp_text value 32p (at 0 1.68) (layer F.Fab)
       (effects (font (size 1 1) (thickness 0.15)))
     )
@@
       (effects (font (size 1 1) (thickness 0.15)))
     )
-    (fp_text value 16p (at 0 1.68) (layer F.Fab)
+    (fp_text value 32p (at 0 1.68) (layer F.Fab)
       (effects (font (size 1 1) (thickness 0.15)))
     )
